File: hardware/WHV_design/WHV_design.kicad_sch (KiCad schematic)
At the start: 31 parts, among them J2 2SMPP-02, U1 74AUC2G08, U10 ${SIM.PARAMS}, U11 ${SIM.PARAMS}, U12 ${SIM.PARAMS}, U13 ${SIM.PARAMS}, U14 ${SIM.PARAMS}, U15 ${SIM.PARAMS}, U16 74AUC2G08, U17 74AHC1G04, U18 74AHC1G86, U2 74AUC2G08, U3 74AUC2G08, U4 74AUC2G08, U5 74AUC2G08, U6 74LVC2G04, U7 74LVC2G04, U8 74LVC1G332, U9 74LVC1G332

Commit message: Mega changes on the schematics and pcb
Parts:
- removed J2: 2SMPP-02, 2SMPP-02_OMR, symbol pressure sensor:2SMPP-02
- removed R1, R10, R11, R12, R2, R3, R4, R5, R6, R7, R8, R9: R, symbol Device:R
- removed U10, U11, U12, U13, U14, U15: ${SIM.PARAMS}, symbol Simulation_SPICE:OPAMP
- removed U16: 74AUC2G08, symbol 74xGxx:74AUC2G08
- removed U17: 74AHC1G04, symbol 74xGxx:74AHC1G04
- removed U18: 74AHC1G86, symbol 74xGxx:74AHC1G86
- added U10, U11, U12, U13, U14, U15, U16, U17: XGZP6859D, Sensor_Pressure:CFSensor_XGZP6859D_7x7mm, symbol Sensor_Pressure:XGZP6859D
- added U18, U19: 74HCT238, symbol 74xx:74HCT238
Connections:
- net +5V: now also U10.2 (VDD), U11.2 (VDD), U12.2 (VDD), U13.2 (VDD), U14.2 (VDD), U15.2 (VDD), U16.2 (VDD), U17.2 (VDD)
- net GND: now also U10.6 (GND), U11.6 (GND), U12.6 (GND), U13.6 (GND), U14.6 (GND), U15.6 (GND), U16.6 (GND), U17.6 (GND), U18.4 (~{E1}), U18.5 (~{E2}), U18.8 (GND), U19.4 (~{E1}), U19.5 (~{E2}), U19.8 (GND)
- net S_0: now also U18.6 (E3)
- net S_1: now also U19.6 (E3)
- new net A0: U18.1 (A0), U19.1 (A0)
- new net A1: U18.2 (A1), U19.2 (A1)
- new net A2: U18.3 (A2), U19.3 (A2)
- new net N0_0: U18.15 (Y0)
- new net N0_1: U19.15 (Y0)
- new net N1_0: U18.14 (Y1)
- new net N1_1: U19.14 (Y1)
- new net N2_0: U18.13 (Y2)
- new net N2_1: U19.13 (Y2)
- new net N3_0: U18.12 (Y3)
- new net N3_1: U19.12 (Y3)
- new net N4_0: U18.11 (Y4)
- new net N4_1: U19.11 (Y4)
- new net N5_0: U18.10 (Y5)
- new net N5_1: U19.10 (Y5)
- new net N6_0: U18.9 (Y6)
- new net N6_1: U19.9 (Y6)
- new net N7_0: U18.7 (Y7)
- new net N7_1: U19.7 (Y7)
- new net SCL_0: U10.5 (SCL)
- new net SCL_1: U11.5 (SCL)
- new net SCL_2: U12.5 (SCL)
- new net SCL_3: U13.5 (SCL)
- new net SCL_4: U14.5 (SCL)
- new net SCL_5: U15.5 (SCL)
- new net SCL_6: U16.5 (SCL)
- new net SCL_7: U17.5 (SCL)
- new net SDA_0: U10.4 (SDA)
- new net SDA_1: U11.4 (SDA)
- new net SDA_2: U12.4 (SDA)
- new net SDA_3: U13.4 (SDA)
- new net SDA_4: U14.4 (SDA)
- new net SDA_5: U15.4 (SDA)
- new net SDA_6: U16.4 (SDA)
- new net SDA_7: U17.4 (SDA)
- no-connect marks 1 -> 0
Other:
- note added: "Fill: 11 Exhaust: 01 Closed:10"
- moved on the sheet: U1A, U1B, U1C, U2A, U2B, U2C, U3A, U3B, U3C, U4A, U4B, U4C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
